File: RoutageBE3A.kicad_pcb (KiCad board)
At the start: 2 copper layers, 110 x 100 mm, 52 parts, among them J2 Conn_01x02, J3 Conn_01x03, Q1 2N2907, Q10 TIP32, Q11 BD138, Q12 TIP31, Q13 2N2222, Q2 2N2907, Q3 2N2907, Q4 2N2222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

Commit message: AvisPlacement
Parts:
- moved Q2 201.0 mm to (62.2, 130.8)
- moved Q1 198.7 mm to (77.7, 128.4)
- moved C4 193.1 mm to (54.6, 100.3)
- moved R3 189.6 mm to (53.3, 134.6), turned to 90 degrees
- moved RV1 174.4 mm to (81.3, 104.1), turned to 180 degrees
- moved C11 172.0 mm to (62.2, 54.6)
- moved R2 171.4 mm to (102.9, 141.0), turned to 90 degrees
- moved Q8 165.7 mm to (94.0, 96.5)
- moved Q3 165.6 mm to (73.7, 114.3), turned to 270 degrees
- moved R1 165.2 mm to (66.0, 137.2), turned to 270 degrees
- moved C5 164.3 mm to (64.8, 94.0), turned to 270 degrees
- moved Q11 159.4 mm to (74.9, 96.5)
- moved Q12 155.3 mm to (68.6, 86.4)
- moved D1 155.2 mm to (97.8, 74.9)
- moved Q4 150.4 mm to (123.2, 130.8), turned to 180 degrees
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