File: RoutageBE3A.kicad_pcb (KiCad board)
At the start: 2 copper layers, 110 x 100 mm, 52 parts, among them J2 Conn_01x02, J3 Conn_01x03, Q1 2N2907, Q10 TIP32, Q11 BD138, Q12 TIP31, Q13 2N2222, Q2 2N2907, Q3 2N2907, Q4 2N2222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

Commit message: Routage1
Parts:
- U1: footprint CmpAmpliAudio:Relay -> CmpAmpliAudioTR:Relais_112LMH2
- moved C10 96.5 mm to (57.1, 67.9), turned to 0 degrees
- moved C8 87.6 mm to (148.6, 66.7), turned to 0 degrees
- moved U1 45.9 mm to (118.1, 92.7), turned to 90 degrees
- moved R11 20.4 mm to (139.7, 70.5), turned to 180 degrees
- moved R12 17.9 mm to (91.4, 70.5), turned to 180 degrees
- moved Q11 6.87 mm to (71.1, 90.8), turned to 180 degrees
- moved Q9 5.68 mm to (139.7, 91.4), turned to 180 degrees
- moved C5 2.84 mm to (66.0, 96.5)
- moved C9 2.29 mm to (143.5, 55.2)
Routing:
- net -12V: track 0.00 -> 75.0 mm
- net GND: track 0.00 -> 29.0 mm
- net /R11-R12: track 0.00 -> 27.9 mm
- net /Q10-R11: track 0.00 -> 21.0 mm
- net /Q11-R12: track 0.00 -> 20.3 mm
- net +12V: track 0.00 -> 13.5 mm
- net /Q9-Q10: track 0.00 -> 5.08 mm
- net /Q11-Q12: track 0.00 -> 4.45 mm

Commit message: Routage2
Parts:
- moved R8 70.1 mm to (73.0, 95.9), turned to 270 degrees
- moved Q6 43.8 mm to (95.2, 106.0), turned to 90 degrees
- moved Q7 15.4 mm to (114.9, 107.3), turned to 90 degrees
- moved R10 14.0 mm to (124.5, 109.9), turned to 0 degrees
- moved R2 13.7 mm to (108.0, 128.3), turned to 270 degrees
- moved RV2 12.8 mm to (132.1, 104.1)
- moved R9 12.0 mm to (100.3, 121.9), turned to 90 degrees
- moved R7 10.9 mm to (91.4, 121.9), turned to 90 degrees
- moved R4 10.3 mm to (81.9, 111.8), turned to 270 degrees
- moved Dz1 10.2 mm to (54.6, 109.2), turned to 270 degrees
- moved R17 10.2 mm to (118.1, 77.5), turned to 270 degrees
- moved C3 9.44 mm to (99.1, 94.6), turned to 180 degrees
- moved Q8 7.65 mm to (86.4, 97.2), turned to 270 degrees
- moved Q4 4.58 mm to (120.7, 127.0), turned to 270 degrees
- moved RV1 4.49 mm to (80.6, 99.7), turned to 90 degrees
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Routing:
- net -12V: track 75.0 -> 344.5 mm
- net +12V: track 13.5 -> 258.6 mm, vias 0 -> 4
- net /R11-R12: track 27.9 -> 155.2 mm, vias 0 -> 1
- net /Q5-Q11: track 0.00 -> 123.8 mm, vias 0 -> 2
- net /Q2-R15: track 0.00 -> 112.5 mm, vias 0 -> 2
- net /Q6-Q9: track 0.00 -> 60.4 mm
- net GND: track 29.0 -> 86.8 mm
- net /C2-sortiediff: track 0.00 -> 49.1 mm
- net /C1-Q1: track 0.00 -> 33.9 mm
- net /U1-J2: track 0.00 -> 32.6 mm
- net /Q6-Q7: track 0.00 -> 30.0 mm
- net /Q1-Q2: track 0.00 -> 26.1 mm
- net /Q5-R6: track 0.00 -> 22.2 mm
- net /R5-Q3: track 0.00 -> 21.9 mm
- net /Q13-R17: track 0.00 -> 21.2 mm
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- added copper zone on B.Cu, net GND
Other:
- board text added: "BOTTOM"
- board text added: "TOP"

Commit message: AvisRoutage1
Routing:
- net GND: track 86.8 -> 6.92 mm
- net /Q5-Q11: track 123.8 -> 118.6 mm
- net /Q2-R15: track 112.5 -> 111.4 mm
