File: RoutageBE3A.sch (KiCad schematic (older format))
At the start: 52 parts, among them J2 Conn_01x02, J3 Conn_01x03, Q1 2N2907, Q10 TIP32, Q11 BD138, Q12 TIP31, Q13 2N2222, Q2 2N2907, Q3 2N2907, Q4 2N2222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

Commit message: AddedFeatures
Parts:
- U1: footprint Relay_THT:Relay_StandexMeder_DIP_LowProfile -> CmpAmpliAudio:Relay
Changed lines of the file:
@@
 encoding utf-8
 Sheet 1 1
-Title ""
-Date ""
-Rev ""
-Comp ""
-Comment1 ""
+Title "Buck 45V vers 24/12V 13A"
+Date "2020-04-12"
+Rev "V0"
+Comp "INSA GEI"
+Comment1 "LERAT MAIER"
 Comment2 ""
 Comment3 ""
@@
 F 0 "U1" V 9467 2900 50  0000 C CNN
 F 1 "Relay_1CT" V 9376 2900 50  0000 C CNN
-F 2 "Relay_THT:Relay_StandexMeder_DIP_LowProfile" H 9350 2850 50  0001 L CNN
+F 2 "CmpAmpliAudio:Relay" H 9350 2850 50  0001 L CNN
 F 3 "https://standexelectronics.com/wp-content/uploads/datasheet_reed_relay_DIP.pdf" H 9000 2900 50  0001 C CNN
 	1    9000 2900

Commit message: Routage1
Parts:
- U1: footprint CmpAmpliAudio:Relay -> CmpAmpliAudioTR:Relais_112LMH2
Changed lines of the file:
@@
 F 0 "U1" V 9467 2900 50  0000 C CNN
 F 1 "Relay_1CT" V 9376 2900 50  0000 C CNN
-F 2 "CmpAmpliAudio:Relay" H 9350 2850 50  0001 L CNN
+F 2 "CmpAmpliAudioTR:Relais_112LMH2" H 9350 2850 50  0001 L CNN
 F 3 "https://standexelectronics.com/wp-content/uploads/datasheet_reed_relay_DIP.pdf" H 9000 2900 50  0001 C CNN
 	1    9000 2900
